Commit message: Updated URDF

File: src/robotont_description/urdf/gen3/base.urdf.xacro (robot description, xacro)
@@ -18,5 +18,5 @@
         <link name="${prefix}base_link">
             <visual>
-                <origin rpy="0 0 ${pi/2}" xyz="0 0 ${frame_elevation}"/>
+                <origin rpy="${-pi / 2} 0 ${pi / 2}" xyz="0 0 ${frame_elevation}"/>
                 <geometry>
                     <mesh filename="package://robotont_description/meshes/gen3/frame_module_pla.STL"/>
@@ -30,5 +30,5 @@
                     <mesh filename="package://robotont_description/meshes/shared/collision_body.STL"/>
                 </geometry>
-                <origin rpy="${pi/2} 0 ${pi/2}" xyz="0 0 ${frame_elevation}"/>
+                <origin rpy="0 0 ${pi / 2}" xyz="0 0 ${frame_elevation}"/>
             </collision>
             <inertial>
@@ -49,5 +49,5 @@
             <origin xyz="0 0 0" rpy="0 0 0"/>
         </joint>
-        <link name="${prefix}base_link_spacers">
+        <!-- <link name="${prefix}base_link_spacers">
             <visual>
                 <origin rpy="0 0 ${pi/2}" xyz="0 0 ${frame_elevation}"/>
@@ -63,6 +63,6 @@
             <parent link="${prefix}base_footprint"/>
             <child link="${prefix}base_link_spacers"/>
-            <origin xyz="0 0 0" rpy="0 0 ${frame_elevation}"/>
-        </joint>
+            <origin xyz="0 0 0" rpy="${pi} ${pi / 2} 0"/>
+        </joint> -->
         <!-- PCB -->
         <link name="${prefix}pcb_link">
@@ -80,5 +80,5 @@
             <parent link="${prefix}base_link"/>
             <child link="${prefix}pcb_link"/>
-            <origin xyz="0.0025 0 ${frame_ground_clearance + pcb_offset}" rpy="0 ${pi / 2} 0"/>
+            <origin xyz="0.0025 0 ${frame_ground_clearance + pcb_offset}" rpy="0 0 0"/>
         </joint>
         <!-- E-button -->
@@ -99,5 +99,5 @@
             <origin
                 xyz="0.0075 0.115 ${frame_ground_clearance + frame_height - e_button_offset}"
-                rpy="${pi / 2} 0 ${pi / 2}"
+                rpy="0 0 ${pi / 2}"
             />
         </joint>
@@ -119,5 +119,5 @@
             <origin
                 xyz="-0.0472 0.111 ${frame_ground_clearance + frame_height - 0.001}"
-                rpy="${pi / 2} 0 ${pi / 2}"
+                rpy="0 0 0"
             />
         </joint>
@@ -139,9 +139,9 @@
             <origin
                 xyz="-0.07 0.12 ${frame_ground_clearance + frame_height - 0.007}"
-                rpy="0 0 0"
+                rpy="${-pi / 2} 0 ${pi / 2}"
             />
         </joint>
         <!-- Battery module -->
-        <link name="${prefix}battery_module_link">
+        <!-- <link name="${prefix}battery_module_link">
             <visual>
                 <geometry>
@@ -159,9 +159,9 @@
             <origin
                 xyz="0.08 0 ${frame_ground_clearance + frame_height + 0.0025}"
-                rpy="${pi / 2} 0 ${pi / 2}"
+                rpy="0 ${pi} ${pi / 2}"
             />
-        </joint>
+        </joint> -->
         <!-- OLED module -->
-        <link name="${prefix}screen_module_link">
+        <!-- <link name="${prefix}screen_module_link">
             <visual>
                 <geometry>
@@ -179,7 +179,7 @@
             <origin
                 xyz="-0.0325 0.1185 ${frame_ground_clearance + frame_height-0.0015}"
-                rpy="0 0 0"
+                rpy="${-pi / 2} 0 ${pi / 2}"
             />
-        </joint>
+        </joint> -->
     </xacro:macro>
 </robot>

File: src/robotont_description/urdf/gen3/motor.urdf.xacro (robot description, xacro)
@@ -35,5 +35,5 @@
             <origin
                 xyz="${distance_from_center * sin(angle) + wheel_center_offset} ${-distance_from_center * cos(angle)} ${ground_clearance}"
-                rpy="${pi/2} 0 ${angle + pi + z_rotation}"
+                rpy="0 0 ${angle + pi + z_rotation}"
             />
         </joint>

File: src/robotont_description/urdf/shared/rim.urdf.xacro (robot description, xacro)
@@ -20,4 +20,5 @@
         <link name="${prefix}rim_${name}_link">
             <visual>
+                <origin xyz="0 0 0" rpy="${pi / 2} 0 0"/>
                 <geometry>
                     <mesh filename="package://robotont_description/meshes/shared/2.75rim.STL"/>
@@ -51,5 +52,5 @@
             <origin
                 xyz="${wheel_center_offset + (wheel_distance * sin(angle))} ${ -wheel_distance * cos(angle)} ${wheel_center_height + wheel_height_offset}"
-                rpy="${pi/2} 0 ${angle + pi}"
+                rpy="${-pi / 2} 0 ${angle + pi}"
             />
             <dynamics damping="0.1"/>
