Commit message: Added nav2, slam, tested in foxglove

File: src/robotont_description/urdf/gen3/robotont.urdf.xacro (robot description, xacro)
@@ -25,4 +25,10 @@
     <xacro:property name="battery_module_color" value="0.26 0.26 0.26 1.0"/>
     <link name="${prefix}base_footprint"/>
+    <link name="${prefix}base_scan"/>
+    <joint name="${prefix}base_scan_joint" type="fixed">
+        <parent link="${prefix}base_link"/>
+        <child link="${prefix}base_scan"/>
+        <origin xyz="0.08 0 0.10" rpy="0 0 0"/>
+    </joint>
     <!-- Frame module -->
     <xacro:base_macro
